Commit message: Some stuff

File: src/motoman/motoman_sda10f_support/urdf/arm_macro.xacro (robot description, xacro)
@@ -108,4 +108,5 @@
 			</visual>
 			<collision>
+				<origin rpy="0 0 0" xyz="0 0 0.0"/>
 				<geometry>
 					<mesh filename="package://motoman_sda10f_support/meshes/sda10f/collision/motoman_axis_t.stl" />
@@ -114,5 +115,19 @@
 			</collision>
 		</link>
-	    <link name="${prefix}link_tool0" />
+	        <link name="${prefix}link_tool0" >
+			<visual>
+				<geometry>
+					<mesh filename="package://motoman_sda10f_support/meshes/sda10f/collision/motoman_axis_t.stl" />
+				</geometry>
+				<material name="blue"/>
+			</visual>
+			<collision>
+				<origin rpy="0 0 0" xyz="0 0 0.0"/>
+				<geometry>
+					<mesh filename="package://motoman_sda10f_support/meshes/sda10f/collision/motoman_axis_t.stl" />
+				</geometry>
+				<material name="yellow"/>
+			</collision>
+		</link>
 		<joint name="${prefix}joint_1_s" type="revolute">
 			<parent link="${parent}"/>
@@ -161,12 +176,12 @@
 			<child link="${prefix}link_7_t"/>
 			<origin xyz="0 0.168 -0.015" rpy="1.57 0 0"/>
-			<axis xyz="0 0 ${-reflect}" />
+			<axis xyz="0 0 ${reflect}" />
 			<limit lower="-3.13" upper="3.13" effort="0" velocity="6.97" />
 		</joint>
-    <joint name="${prefix}joint_tool0" type="fixed" >
-      <origin xyz="0 0 0.0" rpy="0 0 -3.13"/>
-      <parent link="${prefix}link_7_t" />
-      <child link="${prefix}link_tool0" />
-    </joint>
+    		<joint name="${prefix}joint_tool0" type="fixed" >
+      			<origin xyz="0 0.0 -0.15" rpy="0 0 0"/>
+      			<parent link="${prefix}link_7_t" />
+      			<child link="${prefix}link_tool0" />
+    		</joint>
 		<!-- end of joint list -->
 	</xacro:macro>

File: src/motoman/motoman_sda10f_support/urdf/common_torso_macro.xacro (robot description, xacro)
@@ -71,5 +71,4 @@
 			<axis xyz="0 0 1" />
 			<limit lower="-2.9570" upper="2.9570" effort="100" velocity="2.26" />
-			<mimic joint="${prefix}joint_b1" multiplier="1" offset="0"/>
 		</joint>
 		<!-- end of joint list -->

File: src/motoman/motoman_sda10f_support/urdf/sda10f_macro.xacro (robot description, xacro)
@@ -4,9 +4,4 @@
      <xacro:include filename="$(find motoman_sda10f_support)/urdf/arm_macro.xacro" />
      <xacro:include filename="$(find robotiq_2f_c2_gripper_visualization)/urdf/robotiq_c2_model_macro.xacro" />
-     <!-- <xacro:robotiq_c2_model prefix="left_" /> -->
-     <!--
-     <xacro:robotiq_c2_model prefix="left_gripper_" >
-     	<origin xyz="0.0 0.0 0.0" rpy="0 0 0" />
-     </xacro:robotiq_c2_model> -->
      <xacro:macro name="motoman_sda10f" params="prefix">
         <xacro:torso name="${prefix}torso" prefix="${prefix}torso_"/>

Commit message: Pre Removal of Joint

File: src/motoman/motoman_sda10f_support/urdf/arm_macro.xacro (robot description, xacro)
@@ -117,4 +117,5 @@
 	        <link name="${prefix}link_tool0" >
 			<visual>
+				<origin rpy="1.57 0 0" xyz="0 0 0.0"/>
 				<geometry>
 					<mesh filename="package://motoman_sda10f_support/meshes/sda10f/collision/motoman_axis_t.stl" />
@@ -123,5 +124,5 @@
 			</visual>
 			<collision>
-				<origin rpy="0 0 0" xyz="0 0 0.0"/>
+				<origin rpy="1.57 0 0" xyz="0 0 0.0"/>
 				<geometry>
 					<mesh filename="package://motoman_sda10f_support/meshes/sda10f/collision/motoman_axis_t.stl" />
@@ -180,5 +181,5 @@
 		</joint>
     		<joint name="${prefix}joint_tool0" type="fixed" >
-      			<origin xyz="0 0.0 -0.15" rpy="0 0 0"/>
+      			<origin xyz="0 0.1 -0.2	" rpy="1.2 0 0"/>
       			<parent link="${prefix}link_7_t" />
       			<child link="${prefix}link_tool0" />

Commit message: New workspace, New Underactuation with only half of range of motions removed, work on cartesian commands

File: src/motoman/motoman_sda10f_support/urdf/arm_macro.xacro (robot description, xacro)
@@ -181,5 +181,5 @@
 		</joint>
     		<joint name="${prefix}joint_tool0" type="fixed" >
-      			<origin xyz="0 0.1 -0.2	" rpy="1.2 0 0"/>
+      			<origin xyz="0 0.05 -0.25	" rpy="1.0 0 0"/>
       			<parent link="${prefix}link_7_t" />
       			<child link="${prefix}link_tool0" />

File: src/motoman/motoman_sda10f_support/urdf/sda10f_macro.xacro (robot description, xacro)
@@ -7,4 +7,5 @@
      <xacro:macro name="motoman_sda10f" params="prefix">
         <xacro:torso name="${prefix}torso" prefix="${prefix}torso_"/>
+	<!--
         <xacro:motoman_arm name="${prefix}arm_left" prefix="${prefix}arm_left_" parent="${prefix}torso_link_b1" reflect="1">
             <origin xyz="0.09996 0.0275 0.32214" rpy="1.57 0 0" />
@@ -13,6 +14,5 @@
             <origin xyz="0.09996 -0.0275 0.32214" rpy="1.57 0 0" />
         </xacro:motoman_arm>
-	<!--
-	Arm with one degree of freedom removed (7 -> 6) to reduced redundant joint solutions
+	-->
 	<xacro:motoman_under_arm name="${prefix}arm_left" prefix="${prefix}arm_left_" parent="${prefix}torso_link_b1" reflect="1">
             <origin xyz="0.09996 0.0275 0.32214" rpy="1.57 0 0" />
@@ -21,5 +21,4 @@
             <origin xyz="0.09996 -0.0275 0.32214" rpy="1.57 0 0" />
         </xacro:motoman_under_arm>
-	-->
 	<xacro:robotiq_c2_model prefix="${prefix}arm_right_" parent="${prefix}arm_right_link_7_t">
    	</xacro:robotiq_c2_model>

File: src/motoman/motoman_sda10f_support/urdf/under_arm_macro.xacro (robot description, xacro)
@@ -136,5 +136,5 @@
 			<origin xyz="0.09996 ${reflect*0.0275} 0.32214" rpy="1.57 0 ${(reflect-1)*1.57}"/>
 			<axis xyz="0 0 ${-reflect}" />
-			<limit lower="-3.13" upper="3.13" effort="0" velocity="2.95" />
+			<limit lower="0" upper="3.13" effort="0" velocity="2.95" />
 		</joint>
 		<joint name="${prefix}joint_2_l" type="revolute">
@@ -164,5 +164,5 @@
 			<origin xyz="0 0.1936 0.0155" rpy="1.57 0 0"/>
 			<axis xyz="0 0 ${reflect}" />
-			<limit lower="0.0" upper="0.0" effort="0" velocity="3.48" />
+			<limit lower="0" upper="3.13" effort="0" velocity="3.48" />
 		</joint>
 		<joint name="${prefix}joint_6_b" type="revolute">
@@ -181,5 +181,5 @@
 		</joint>
     		<joint name="${prefix}joint_tool0" type="fixed" >
-      			<origin xyz="0 0.1 -0.2	" rpy="1.2 0 0"/>
+      			<origin xyz="0 0.05 -0.25	" rpy="1.0 0 0"/>
       			<parent link="${prefix}link_7_t" />
       			<child link="${prefix}link_tool0" />

Commit message: Updated Underactuated arm for velocity and such

File: src/motoman/motoman_sda10f_support/urdf/arm_macro.xacro (robot description, xacro)
@@ -181,5 +181,6 @@
 		</joint>
     		<joint name="${prefix}joint_tool0" type="fixed" >
-      			<origin xyz="0 0.05 -0.25	" rpy="1.0 0 0"/>
+      			<origin xyz="0 0.0 -0.15	" rpy="0 0 1.5705"/>
+			<!--<origin xyz="0 0.05 -0.25	" rpy="0 0 0"/>-->
       			<parent link="${prefix}link_7_t" />
       			<child link="${prefix}link_tool0" />

File: src/motoman/motoman_sda10f_support/urdf/sda10f_macro.xacro (robot description, xacro)
@@ -11,14 +11,16 @@
             <origin xyz="0.09996 0.0275 0.32214" rpy="1.57 0 0" />
         </xacro:motoman_arm>
+	-->
 	<xacro:motoman_arm name="${prefix}arm_right" prefix="${prefix}arm_right_" parent="${prefix}torso_link_b1" reflect="-1">
             <origin xyz="0.09996 -0.0275 0.32214" rpy="1.57 0 0" />
         </xacro:motoman_arm>
-	-->
 	<xacro:motoman_under_arm name="${prefix}arm_left" prefix="${prefix}arm_left_" parent="${prefix}torso_link_b1" reflect="1">
             <origin xyz="0.09996 0.0275 0.32214" rpy="1.57 0 0" />
         </xacro:motoman_under_arm>
+	<!--
 	<xacro:motoman_under_arm name="${prefix}arm_right" prefix="${prefix}arm_right_" parent="${prefix}torso_link_b1" reflect="-1">
             <origin xyz="0.09996 -0.0275 0.32214" rpy="1.57 0 0" />
         </xacro:motoman_under_arm>
+	-->
 	<xacro:robotiq_c2_model prefix="${prefix}arm_right_" parent="${prefix}arm_right_link_7_t">
    	</xacro:robotiq_c2_model>

File: src/motoman/motoman_sda10f_support/urdf/under_arm_macro.xacro (robot description, xacro)
@@ -1,3 +1,8 @@
 <?xml version="1.0" ?>
+<!--
+     This Macro Contains a version of the arm with joints and velocities constrained to make testing easier and safer
+     It will reduce the number of solutions to one for most cases in the goal center of the robot's workspace but will
+     also reduce the size of the workspace (such as removing the area above the robot as accessable).
+-->
 <robot xmlns:xacro="http://ros.org/wiki/xacro">
 	<xacro:macro name="motoman_under_arm" params="name prefix parent *origin reflect">
@@ -136,5 +141,6 @@
 			<origin xyz="0.09996 ${reflect*0.0275} 0.32214" rpy="1.57 0 ${(reflect-1)*1.57}"/>
 			<axis xyz="0 0 ${-reflect}" />
-			<limit lower="0" upper="3.13" effort="0" velocity="2.95" />
+			<limit lower="-3.13" upper="0" effort="0" velocity="1" />
+		<!--	<limit lower="-3.13" upper="0" effort="0" velocity="2.95" /> -->
 		</joint>
 		<joint name="${prefix}joint_2_l" type="revolute">
@@ -143,5 +149,6 @@
 			<origin xyz="0 0.0577 -0.2255" rpy="-1.57 0 0"/>
 			<axis xyz="0 0 ${-reflect}" />
-			<limit lower="-1.90" upper="1.90" effort="0" velocity="2.95" />
+			<limit lower="0" upper="1.90" effort="0" velocity="1" />
+		<!--	<limit lower="-1.90"upper="1.90" effort="0" velocity="2.95" />	-->
 		</joint>
 		<joint name="${prefix}joint_3_e" type="revolute">
@@ -150,5 +157,6 @@
 			<origin xyz="0 0.1690 -0.0454" rpy="1.57 0 0"/>
 			<axis xyz="0 0 ${-reflect}" />
-			<limit lower="-2.95" upper="2.95" effort="0" velocity="2.95" />
+			<limit lower="-1.6" upper="1.6" effort="0" velocity="1" />
+		<!--	<limit lower="-2.95" upper="2.95" effort="0" velocity="2.95" /> -->
 		</joint>
 		<joint name="${prefix}joint_4_u" type="revolute">
@@ -157,5 +165,6 @@
 			<origin xyz="0 -0.0085 -0.181" rpy="-1.57 0 0"/>
 			<axis xyz="0 0 ${reflect}" />
-			<limit lower="-2.36" upper="2.36" effort="0" velocity="2.95" />
+			<limit lower="0" upper="2.36" effort="0" velocity="1" />
+		<!--	<limit lower="-2.36" upper="2.36" effort="0" velocity="2.95" /> -->
 		</joint>
 		<joint name="${prefix}joint_5_r" type="revolute">
@@ -164,5 +173,6 @@
 			<origin xyz="0 0.1936 0.0155" rpy="1.57 0 0"/>
 			<axis xyz="0 0 ${reflect}" />
-			<limit lower="0" upper="3.13" effort="0" velocity="3.48" />
+			<limit lower="-3.13" upper="3.13" effort="0" velocity="1.5" />
+		<!--	<limit lower="-3.13" upper="3.13" effort="0" velocity="3.48" /> -->
 		</joint>
 		<joint name="${prefix}joint_6_b" type="revolute">
@@ -171,5 +181,6 @@
 			<origin xyz="0 0.0080 -0.155" rpy="-1.57 0 0"/>
 			<axis xyz="0 0 ${reflect}" />
-			<limit lower="-1.90" upper="1.90" effort="0" velocity="3.48" />
+			<limit lower="-1.90" upper="0" effort="0" velocity="1.5" />
+		<!--	<limit lower="-1.90" upper="1.90" effort="0" velocity="3.48" /> -->
 		</joint>
 		<joint name="${prefix}joint_7_t" type="revolute">
@@ -178,5 +189,6 @@
 			<origin xyz="0 0.168 -0.015" rpy="1.57 0 0"/>
 			<axis xyz="0 0 ${reflect}" />
-			<limit lower="-3.13" upper="3.13" effort="0" velocity="6.97" />
+			<limit lower="-3.13" upper="3.13" effort="0" velocity="3" />
+		<!--	<limit lower="-3.13" upper="0" effort="0" velocity="6.97" />	-->
 		</joint>
     		<joint name="${prefix}joint_tool0" type="fixed" >

Commit message: pre trajectory full planning commit

File: src/motoman/motoman_sda10f_support/urdf/arm_macro.xacro (robot description, xacro)
@@ -181,6 +181,6 @@
 		</joint>
     		<joint name="${prefix}joint_tool0" type="fixed" >
-      			<origin xyz="0 0.0 -0.15	" rpy="0 0 1.5705"/>
-			<!--<origin xyz="0 0.05 -0.25	" rpy="0 0 0"/>-->
+      			<!-- <origin xyz="0 0.0 -0.15	" rpy="0 0 1.5705"/> -->
+			<origin xyz="0 0.05 -0.25" rpy="1 0 0"/>
       			<parent link="${prefix}link_7_t" />
       			<child link="${prefix}link_tool0" />

File: src/motoman/motoman_sda10f_support/urdf/sda10f_macro.xacro (robot description, xacro)
@@ -7,15 +7,15 @@
      <xacro:macro name="motoman_sda10f" params="prefix">
         <xacro:torso name="${prefix}torso" prefix="${prefix}torso_"/>
-	<!--
         <xacro:motoman_arm name="${prefix}arm_left" prefix="${prefix}arm_left_" parent="${prefix}torso_link_b1" reflect="1">
             <origin xyz="0.09996 0.0275 0.32214" rpy="1.57 0 0" />
         </xacro:motoman_arm>
-	-->
 	<xacro:motoman_arm name="${prefix}arm_right" prefix="${prefix}arm_right_" parent="${prefix}torso_link_b1" reflect="-1">
             <origin xyz="0.09996 -0.0275 0.32214" rpy="1.57 0 0" />
         </xacro:motoman_arm>
+	<!--
 	<xacro:motoman_under_arm name="${prefix}arm_left" prefix="${prefix}arm_left_" parent="${prefix}torso_link_b1" reflect="1">
             <origin xyz="0.09996 0.0275 0.32214" rpy="1.57 0 0" />
         </xacro:motoman_under_arm>
+	-->
 	<!--
 	<xacro:motoman_under_arm name="${prefix}arm_right" prefix="${prefix}arm_right_" parent="${prefix}torso_link_b1" reflect="-1">

File: src/motoman/motoman_sda10f_support/urdf/under_arm_macro.xacro (robot description, xacro)
@@ -173,5 +173,5 @@
 			<origin xyz="0 0.1936 0.0155" rpy="1.57 0 0"/>
 			<axis xyz="0 0 ${reflect}" />
-			<limit lower="-3.13" upper="3.13" effort="0" velocity="1.5" />
+			<limit lower="-1.6" upper="1.6" effort="0" velocity="1.5" />
 		<!--	<limit lower="-3.13" upper="3.13" effort="0" velocity="3.48" /> -->
 		</joint>
@@ -189,6 +189,6 @@
 			<origin xyz="0 0.168 -0.015" rpy="1.57 0 0"/>
 			<axis xyz="0 0 ${reflect}" />
-			<limit lower="-3.13" upper="3.13" effort="0" velocity="3" />
-		<!--	<limit lower="-3.13" upper="0" effort="0" velocity="6.97" />	-->
+			<limit lower="-3.13" upper="0" effort="0" velocity="3" />
+		<!--	<limit lower="-3.13" upper="3.13" effort="0" velocity="6.97" />	-->
 		</joint>
     		<joint name="${prefix}joint_tool0" type="fixed" >

Commit message: Vision Relignment working

File: src/motoman/motoman_sda10f_support/urdf/arm_macro.xacro (robot description, xacro)
@@ -182,5 +182,5 @@
     		<joint name="${prefix}joint_tool0" type="fixed" >
       			<!-- <origin xyz="0 0.0 -0.15	" rpy="0 0 1.5705"/> -->
-			<origin xyz="0 0.05 -0.25" rpy="1 0 0"/>
+			<origin xyz="-0.07 0.05 -0.25" rpy="0.8 0 0"/>
       			<parent link="${prefix}link_7_t" />
       			<child link="${prefix}link_tool0" />

Commit message: Pick and Allign

File: src/motoman/motoman_sda10f_support/urdf/arm_macro.xacro (robot description, xacro)
@@ -182,5 +182,6 @@
     		<joint name="${prefix}joint_tool0" type="fixed" >
       			<!-- <origin xyz="0 0.0 -0.15	" rpy="0 0 1.5705"/> -->
-			<origin xyz="-0.07 0.05 -0.25" rpy="0.8 0 0"/>
+			<!-- <origin xyz="-0.07 0.05 -0.25" rpy="0.8 0 0"/> < Used for original alligment testing  -->
+			<origin xyz="0.0 0.05 -0.25" rpy="0.65 0 0"/>
       			<parent link="${prefix}link_7_t" />
       			<child link="${prefix}link_tool0" />

Commit message: cleaned up code

File: src/motoman/motoman_sda10f_support/urdf/arm_macro.xacro (robot description, xacro)
@@ -183,5 +183,5 @@
       			<!-- <origin xyz="0 0.0 -0.15	" rpy="0 0 1.5705"/> -->
 			<!-- <origin xyz="-0.07 0.05 -0.25" rpy="0.8 0 0"/> < Used for original alligment testing  -->
-			<origin xyz="0.0 0.05 -0.25" rpy="0.65 0 0"/>
+			<origin xyz="0.0 0.05 -0.25" rpy="0.65	 0 0"/>
       			<parent link="${prefix}link_7_t" />
       			<child link="${prefix}link_tool0" />

Commit message: more vision

File: src/motoman/motoman_sda10f_support/urdf/arm_macro.xacro (robot description, xacro)
@@ -116,4 +116,36 @@
 		</link>
 	        <link name="${prefix}link_tool0" >
+			<visual>
+				<origin rpy="1.57 0 0" xyz="0 0 0.0"/>
+				<geometry>
+					<mesh filename="package://motoman_sda10f_support/meshes/sda10f/collision/motoman_axis_t.stl" />
+				</geometry>
+				<material name="blue"/>
+			</visual>
+			<collision>
+				<origin rpy="1.57 0 0" xyz="0 0 0.0"/>
+				<geometry>
+					<mesh filename="package://motoman_sda10f_support/meshes/sda10f/collision/motoman_axis_t.stl" />
+				</geometry>
+				<material name="yellow"/>
+			</collision>
+		</link>
+		<link name="${prefix}link_leftN" >
+			<visual>
+				<origin rpy="1.57 0 0" xyz="0 0 0.0"/>
+				<geometry>
+					<mesh filename="package://motoman_sda10f_support/meshes/sda10f/collision/motoman_axis_t.stl" />
+				</geometry>
+				<material name="blue"/>
+			</visual>
+			<collision>
+				<origin rpy="0 0 0" xyz="0 0 0.0"/>
+				<geometry>
+					<mesh filename="package://motoman_sda10f_support/meshes/sda10f/collision/motoman_axis_t.stl" />
+				</geometry>
+				<material name="yellow"/>
+			</collision>
+		</link>
+		<link name="${prefix}link_rightN" >
 			<visual>
 				<origin rpy="1.57 0 0" xyz="0 0 0.0"/>
@@ -183,7 +215,17 @@
       			<!-- <origin xyz="0 0.0 -0.15	" rpy="0 0 1.5705"/> -->
 			<!-- <origin xyz="-0.07 0.05 -0.25" rpy="0.8 0 0"/> < Used for original alligment testing  -->
-			<origin xyz="0.0 0.05 -0.25" rpy="0.65	 0 0"/>
+			<origin xyz="0.0 0.05 -0.30" rpy="0.65	 0 0"/>
       			<parent link="${prefix}link_7_t" />
       			<child link="${prefix}link_tool0" />
+    		</joint>
+		<joint name="${prefix}joint_leftN" type="fixed" >
+			<origin xyz="-0.05 0.0 0.0" rpy="0 0 0"/>
+      			<parent link="${prefix}link_tool0" />
+      			<child link="${prefix}link_leftN" />
+    		</joint>
+		<joint name="${prefix}joint_rightN" type="fixed" >
+			<origin xyz="0.05 0.0 0.0" rpy="0 0 0"/>
+      			<parent link="${prefix}link_tool0" />
+      			<child link="${prefix}link_rightN" />
     		</joint>
 		<!-- end of joint list -->

Commit message: Remade Remade Vision

File: src/motoman/motoman_sda10f_support/urdf/arm_macro.xacro (robot description, xacro)
@@ -131,4 +131,5 @@
 			</collision>
 		</link>
+	<!--
 		<link name="${prefix}link_leftN" >
 			<visual>
@@ -163,4 +164,5 @@
 			</collision>
 		</link>
+	-->
 		<joint name="${prefix}joint_1_s" type="revolute">
 			<parent link="${parent}"/>
@@ -218,5 +220,6 @@
       			<parent link="${prefix}link_7_t" />
       			<child link="${prefix}link_tool0" />
-    		</joint>
+		</joint>
+		<!--
 		<joint name="${prefix}joint_leftN" type="fixed" >
 			<origin xyz="-0.05 0.0 0.0" rpy="0 0 0"/>
@@ -229,4 +232,5 @@
       			<child link="${prefix}link_rightN" />
     		</joint>
+		-->
 		<!-- end of joint list -->
 	</xacro:macro>

Commit message: Nert

File: src/motoman/motoman_sda10f_support/urdf/arm_macro.xacro (robot description, xacro)
@@ -131,5 +131,4 @@
 			</collision>
 		</link>
-	<!--
 		<link name="${prefix}link_leftN" >
 			<visual>
@@ -164,5 +163,4 @@
 			</collision>
 		</link>
-	-->
 		<joint name="${prefix}joint_1_s" type="revolute">
 			<parent link="${parent}"/>
@@ -217,9 +215,9 @@
       			<!-- <origin xyz="0 0.0 -0.15	" rpy="0 0 1.5705"/> -->
 			<!-- <origin xyz="-0.07 0.05 -0.25" rpy="0.8 0 0"/> < Used for original alligment testing  -->
-			<origin xyz="0.0 0.05 -0.30" rpy="0.65	 0 0"/>
+			<!-- <origin xyz="0.0 0.05 -0.30 rpy="0.8 0 0"/> < Value 8/8/19  -->
+			<origin xyz="0.0 0.05 -0.28" rpy="0.65	 0 0"/>
       			<parent link="${prefix}link_7_t" />
       			<child link="${prefix}link_tool0" />
 		</joint>
-		<!--
 		<joint name="${prefix}joint_leftN" type="fixed" >
 			<origin xyz="-0.05 0.0 0.0" rpy="0 0 0"/>
@@ -228,9 +226,8 @@
     		</joint>
 		<joint name="${prefix}joint_rightN" type="fixed" >
-			<origin xyz="0.05 0.0 0.0" rpy="0 0 0"/>
-      			<parent link="${prefix}link_tool0" />
+			<origin xyz="0.1 0.0 0.0" rpy="0 0 0"/>
+      			<parent link="${prefix}link_leftN" />
       			<child link="${prefix}link_rightN" />
     		</joint>
-		-->
 		<!-- end of joint list -->
 	</xacro:macro>

Commit message: Visapp Paper

File: src/motoman/motoman_sda10f_support/urdf/arm_macro.xacro (robot description, xacro)
@@ -216,5 +216,5 @@
 			<!-- <origin xyz="-0.07 0.05 -0.25" rpy="0.8 0 0"/> < Used for original alligment testing  -->
 			<!-- <origin xyz="0.0 0.05 -0.30 rpy="0.8 0 0"/> < Value 8/8/19  -->
-			<origin xyz="0.0 0.05 -0.28" rpy="0.65	 0 0"/>
+			<origin xyz="0.0 0.05 -0.28" rpy="0.68	 0 0"/>
       			<parent link="${prefix}link_7_t" />
       			<child link="${prefix}link_tool0" />
